File: PCB/main/chu_main.kicad_pcb (KiCad board)
At the start: 2 copper layers, 290 x 100 mm, 83 parts, among them K1 Conn_01x01_Female, K10 Conn_01x01_Female, K11 Conn_01x01_Female, K12 Conn_01x01_Female, K13 Conn_01x01_Female, K14 Conn_01x01_Female, K15 Conn_01x01_Female, K16 Conn_01x01_Female, K17 Conn_01x01_Female, K18 Conn_01x01_Female, K19 Conn_01x01_Female, K2 Conn_01x01_Female, K20 Conn_01x01_Female, K21 Conn_01x01_Female, K22 Conn_01x01_Female, K23 Conn_01x01_Female, K24 Conn_01x01_Female, K25 Conn_01x01_Female, K26 Conn_01x01_Female, K27 Conn_01x01_Female, K28 Conn_01x01_Female, K29 Conn_01x01_Female, K3 Conn_01x01_Female, K30 Conn_01x01_Female, K31 Conn_01x01_Female, K32 Conn_01x01_Female, K4 Conn_01x01_Female, K5 Conn_01x01_Female, K6 Conn_01x01_Female, K7 Conn_01x01_Female, K8 Conn_01x01_Female, K9 Conn_01x01_Female, U1 Pico, U3 MPR121QR2_BOARD, U4 MPR121QR2_BOARD, U5 MPR121QR2_BOARD, U8 SN74LV1T34DBV

Commit message: Some updates (keypad, IR sensor firmware)
Parts:
- added IR1: Conn_01x06, chu_main:GP2Y0E03, F.Cu at (244.2, 145.1)
- added IR2: Conn_01x06, chu_main:GP2Y0E03, F.Cu at (174.2, 145.1)
- added IR3: Conn_01x06, chu_main:GP2Y0E03, F.Cu at (86.2, 151.1)
- added IR4: Conn_01x06, chu_main:GP2Y0E03, F.Cu at (342.2, 151.1)
- added IR5: Conn_01x06, chu_main:GP2Y0E03, F.Cu at (254.2, 145.1)
- added U0: ChuAcrylic, chu_main:ChuAcrylic, F.Cu at (214.2, 94.6)
- added U2: PCA9548APW, Package_SO:TSSOP-24_4.4x7.8mm_P0.65mm, B.Cu at (309.2, 143.3)
- added X1: GP2Y0E03_REAL, chu_main:GP2Y0E03_REAL, F.Cu at (75.2, 134.1)
- added X2: GP2Y0E03_REAL, chu_main:GP2Y0E03_REAL, F.Cu at (144.2, 146.1)
- added X3: GP2Y0E03_REAL, chu_main:GP2Y0E03_REAL, F.Cu at (214.2, 146.1)
- added X4: GP2Y0E03_REAL, chu_main:GP2Y0E03_REAL, F.Cu at (284.2, 146.1)
- added X5: GP2Y0E03_REAL, chu_main:GP2Y0E03_REAL, F.Cu at (353.2, 134.1)
- C1, C2, C3, C4, C5, C6, C7, R20, R21, R4, U8: moved to B.Cu
- moved R4 212.5 mm to (316.7, 147.1), turned to 180 degrees
- moved U8 202.5 mm to (311.7, 152.1), turned to 180 degrees
- moved C4 86.2 mm to (253.0, 155.8), turned to 180 degrees
- moved C5 71.2 mm to (246.1, 127.1), turned to 180 degrees
- moved C2 62.5 mm to (241.7, 127.1), turned to 180 degrees
- moved C1 59.6 mm to (242.2, 155.8), turned to 180 degrees
- moved C3 54.0 mm to (237.5, 156.1), turned to 180 degrees
- moved C7 22.2 mm to (230.3, 155.6), turned to 180 degrees
- moved SCR3 15.3 mm to (74.2, 144.1)
- moved SCR4 15.3 mm to (354.2, 144.1)
- moved R20 15.2 mm to (340.4, 114.8), turned to 180 degrees
- moved C6 14.5 mm to (226.0, 155.6), turned to 180 degrees
- moved U3 11.0 mm to (134.2, 135.1)
- moved U4 11.0 mm to (214.2, 135.1)
- moved U5 9.80 mm to (264.2, 135.1)
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Other:
- board size 290 x 100 mm -> 300 x 100 mm

Commit message: Layout progress 40%
Parts:
- added D32: WS2812B_Unified, chu_main:WS2812B-2835, F.Cu at (354.7, 137.6)
- added D33: WS2812B_Unified, chu_main:WS2812B-2835, F.Cu at (284.2, 149.8)
- added D34: WS2812B_Unified, chu_main:WS2812B-2835, F.Cu at (214.2, 149.8)
- added D35: WS2812B_Unified, chu_main:WS2812B-2835, F.Cu at (144.2, 149.8)
- added D36: WS2812B_Unified, chu_main:WS2812B-2835, F.Cu at (73.7, 137.6)
- moved USB1 278.1 mm to (74.2, 114.1), turned to 70.75 degrees
- moved R4 236.6 mm to (86.2, 94.0)
- moved U8 229.8 mm to (88.3, 98.0)
- moved U1 203.0 mm to (106.2, 142.1), turned to -90 degrees
- moved IR3 168.8 mm to (254.2, 135.1), turned to 180 degrees
- moved IR1 130.2 mm to (114.2, 152.1), turned to 0 degrees
- moved U2 111.0 mm to (198.2, 146.1), turned to 0 degrees
- moved IR4 96.0 mm to (246.2, 152.1)
- moved IR5 64.4 mm to (318.2, 152.1), turned to 0 degrees
- moved U5 38.0 mm to (302.2, 135.1)
- moved C2 36.3 mm to (259.0, 159.0)
- moved C5 36.3 mm to (263.4, 159.0)
- moved U3 16.0 mm to (150.2, 135.1)
- moved IR2 10.6 mm to (182.2, 152.1), turned to 0 degrees
- moved U4 10.0 mm to (224.2, 135.1)
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Routing:
- net +5V: track 0.00 -> 356.8 mm
- net Net-(K1-Pad1): track 0.00 -> 78.5 mm, vias 0 -> 1
- net Net-(K23-Pad1): track 0.00 -> 76.7 mm, vias 0 -> 1
- net Net-(K3-Pad1): track 0.00 -> 68.9 mm, vias 0 -> 1
- net Net-(K31-Pad1): track 0.00 -> 67.9 mm, vias 0 -> 1
- net Net-(K21-Pad1): track 0.00 -> 67.5 mm, vias 0 -> 1
- net Net-(K13-Pad1): track 0.00 -> 66.5 mm, vias 0 -> 1
- net Net-(K11-Pad1): track 0.00 -> 64.6 mm, vias 0 -> 1
- net Net-(K5-Pad1): track 0.00 -> 64.5 mm, vias 0 -> 1
- net Net-(K29-Pad1): track 0.00 -> 63.0 mm, vias 0 -> 1
- net Net-(K19-Pad1): track 0.00 -> 62.1 mm, vias 0 -> 1
- net Net-(K25-Pad1): track 0.00 -> 60.1 mm, vias 0 -> 1
- net Net-(K15-Pad1): track 0.00 -> 58.5 mm, vias 0 -> 1
- net Net-(K9-Pad1): track 0.00 -> 57.7 mm, vias 0 -> 1
- net Net-(K7-Pad1): track 0.00 -> 56.2 mm, vias 0 -> 1
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Other:
- board size 300 x 100 mm -> 294 x 100 mm

Commit message: Layoug progress 70%
Parts:
- added R10: 4.7K, Resistor_SMD:R_0603_1608Metric, B.Cu at (254.8, 147.2)
- added R11: 4.7K, Resistor_SMD:R_0603_1608Metric, B.Cu at (252.8, 147.2)
- added R12: 4.7K, Resistor_SMD:R_0603_1608Metric, B.Cu at (327.4, 150.9)
- added R13: 4.7K, Resistor_SMD:R_0603_1608Metric, B.Cu at (329.3, 150.9)
- added R4: 4.7K, Resistor_SMD:R_0603_1608Metric, B.Cu at (184.4, 142.5)
- added R5: 4.7K, Resistor_SMD:R_0603_1608Metric, B.Cu at (182.6, 142.5)
- added R6: 4.7K, Resistor_SMD:R_0603_1608Metric, B.Cu at (183.2, 149.0)
- added R7: 4.7K, Resistor_SMD:R_0603_1608Metric, B.Cu at (181.4, 149.0)
- added R8: 4.7K, Resistor_SMD:R_0603_1608Metric, B.Cu at (253.5, 137.7)
- added R9: 4.7K, Resistor_SMD:R_0603_1608Metric, B.Cu at (255.5, 137.7)
- U1: footprint chu_main:RPi_Pico_SMD_Pins -> chu_main:RPi_Pico_SMD_Pins_Strip
- moved R2 257.2 mm to (86.4, 115.8), turned to 0 degrees
- moved R1 254.7 mm to (85.8, 118.7), turned to 0 degrees
- moved C5 33.2 mm to (232.6, 171.5)
- moved C7 33.2 mm to (199.5, 168.1)
- moved C1 33.2 mm to (211.4, 168.3)
- moved C2 33.2 mm to (228.3, 171.5)
- moved C3 33.2 mm to (206.7, 168.6)
- moved C4 33.2 mm to (222.2, 168.3)
- moved C6 33.2 mm to (195.2, 168.1)
- moved U8 8.93 mm to (89.5, 89.2), turned to 90 degrees
- moved R3 5.22 mm to (87.0, 88.9), turned to -90 degrees
- moved U2 3.16 mm to (199.2, 143.1), turned to 180 degrees
- moved IR1 2.00 mm to (114.2, 150.1)
- moved IR2 2.00 mm to (182.2, 150.1)
- moved IR4 2.00 mm to (246.2, 150.1)
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- renumbered R20 to R1, R21 to R2, R4 to R3
Connections:
- IR1 pad 5: Net-(IR1-Pad5) -> /SCL_1
- IR1 pad 6: Net-(IR1-Pad6) -> /SDA_1
- IR2 pad 5: Net-(IR2-Pad5) -> /SCL_2
- IR2 pad 6: Net-(IR2-Pad6) -> /SDA_2
- IR3 pad 5: Net-(IR3-Pad5) -> /SCL_3
- IR3 pad 6: Net-(IR3-Pad6) -> /SDA_3
- IR4 pad 5: Net-(IR4-Pad5) -> /SCL_4
- IR4 pad 6: Net-(IR4-Pad6) -> /SDA_4
- IR5 pad 5: Net-(IR5-Pad5) -> /SCL_5
- IR5 pad 6: Net-(IR5-Pad6) -> /SDA_5
- R3 pad 2: Net-(R4-Pad2) -> Net-(R3-Pad2)
- U1 pad 10: /SCL -> unconnected-(U1-Pad10)
- U1 pad 17: Net-(R4-Pad2) -> unconnected-(U1-Pad17)
- U1 pad 21: unconnected-(U1-Pad21) -> /SDA
- U1 pad 22: unconnected-(U1-Pad22) -> /SCL
- U1 pad 25: unconnected-(U1-Pad25) -> Net-(U2-Pad3)
- U1 pad 4: unconnected-(U1-Pad4) -> Net-(R3-Pad2)
- U1 pad 9: /SDA -> unconnected-(U1-Pad9)
- U2 pad 1: unconnected-(U2-Pad1) -> GND
- U2 pad 12: unconnected-(U2-Pad12) -> GND
- U2 pad 13: Net-(IR4-Pad6) -> /SDA_2
- U2 pad 14: Net-(IR4-Pad5) -> /SCL_2
- U2 pad 15: Net-(IR5-Pad6) -> /SDA_1
- U2 pad 16: Net-(IR5-Pad5) -> /SCL_1
- U2 pad 2: unconnected-(U2-Pad2) -> GND
- U2 pad 21: unconnected-(U2-Pad21) -> GND
- U2 pad 22: unconnected-(U2-Pad22) -> /SCL
- U2 pad 23: unconnected-(U2-Pad23) -> /SDA
- U2 pad 24: unconnected-(U2-Pad24) -> +3V3
- U2 pad 3: unconnected-(U2-Pad3) -> Net-(U2-Pad3)
- U2 pad 4: Net-(IR1-Pad6) -> /SDA_3
- U2 pad 5: Net-(IR1-Pad5) -> /SCL_3
- U2 pad 6: Net-(IR2-Pad6) -> /SDA_5
- U2 pad 7: Net-(IR2-Pad5) -> /SCL_5
- U2 pad 8: Net-(IR3-Pad6) -> /SDA_4
- U2 pad 9: Net-(IR3-Pad5) -> /SCL_4
- U8 pad 2: Net-(R4-Pad2) -> Net-(R3-Pad2)
Routing:
- net GND: track 0.00 -> 818.6 mm, vias 0 -> 2
- net +3V3: track 0.00 -> 424.8 mm, vias 0 -> 5
- net +5V: track 356.8 -> 754.7 mm, vias 0 -> 5
- net /SCL: track 0.00 -> 204.6 mm, vias 0 -> 3
- net /SDA: track 0.00 -> 203.1 mm, vias 0 -> 3
- net /SDA_5: track 0.00 -> 132.0 mm, vias 0 -> 1
- net /SCL_5: track 0.00 -> 129.7 mm, vias 0 -> 1
- net Net-(U2-Pad3): track 0.00 -> 98.1 mm
- net Net-(D31-PadO): track 0.00 -> 90.2 mm
- net Net-(D35-PadO): track 0.00 -> 85.5 mm
- net /SCL_1: track 0.00 -> 85.0 mm, vias 0 -> 1
- net /SDA_1: track 0.00 -> 83.7 mm, vias 0 -> 3
- net Net-(D32-PadO): track 0.00 -> 78.2 mm
- net Net-(D34-PadO): track 0.00 -> 75.3 mm
- net Net-(D33-PadO): track 0.00 -> 74.9 mm
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- added copper zone on B.Cu, net GND
- added copper zone on F.Cu, net GND
