File: PCB/main/chu_main.kicad_pcb (KiCad board)
At the start: 2 copper layers, 294 x 100 mm, 112 parts, among them J1 Conn_01x04, K1 Conn_01x01_Female, K10 Conn_01x01_Female, K11 Conn_01x01_Female, K12 Conn_01x01_Female, K13 Conn_01x01_Female, K14 Conn_01x01_Female, K15 Conn_01x01_Female, K16 Conn_01x01_Female, K17 Conn_01x01_Female, K18 Conn_01x01_Female, K19 Conn_01x01_Female, K2 Conn_01x01_Female, K20 Conn_01x01_Female, K21 Conn_01x01_Female, K22 Conn_01x01_Female, K23 Conn_01x01_Female, K24 Conn_01x01_Female, K25 Conn_01x01_Female, K26 Conn_01x01_Female, K27 Conn_01x01_Female, K28 Conn_01x01_Female, K29 Conn_01x01_Female, K3 Conn_01x01_Female, K30 Conn_01x01_Female, K31 Conn_01x01_Female, K32 Conn_01x01_Female, K4 Conn_01x01_Female, K5 Conn_01x01_Female, K6 Conn_01x01_Female, K7 Conn_01x01_Female, K8 Conn_01x01_Female, K9 Conn_01x01_Female, U0 ChuAcrylic, U1 Pico, U2 PCA9548APW, U3 MPR121QR2_BOARD, U4 MPR121QR2_BOARD, U5 MPR121QR2_BOARD, U8 SN74LV1T34DBV, X1 GP2Y0E03_REAL, X2 GP2Y0E03_REAL, X3 GP2Y0E03_REAL, X4 GP2Y0E03_REAL, X5 GP2Y0E03_REAL

Commit message: Chu main PCB v1.6
Parts:
- removed R3: 10, Resistor_SMD:R_0603_1608Metric
- removed U8: SN74LV1T34DBV, chu_main:SOT-23-5_Jumper
- added SW1: SPST_EVQP4, chu_main:SW_EVQ-P46B3M, B.Cu at (351.8, 111.1)
- added SW2: SPST_EVQP4, chu_main:SW_EVQ-P46B3M, B.Cu at (348.3, 101.1)
- added SW3: SPST_EVQP4, chu_main:SW_EVQ-P46B3M, B.Cu at (344.8, 91.1)
- PN532: renamed from J1; value Conn_01x04 -> TOF_I2C; footprint chu_main:PN532 -> chu_main:SH1.0_4P_Solder_Combo
- R1, R10, R11, R12, R13, R2, R4, R5, R6, R7, R8, R9: footprint Resistor_SMD:R_0603_1608Metric -> Resistor_SMD:R_0603_1608Metric_Pad0.98x0.95mm_HandSolder
- TOF1: renamed from IR1; value Conn_01x06 -> TOF_I2C; footprint chu_main:GP2Y0E03 -> chu_main:SH1.0_4P_Solder_Combo
- TOF2: renamed from IR2; value Conn_01x06 -> TOF_I2C; footprint chu_main:GP2Y0E03 -> chu_main:SH1.0_4P_Solder_Combo
- TOF3: renamed from IR3; value Conn_01x06 -> TOF_I2C; footprint chu_main:GP2Y0E03 -> chu_main:SH1.0_4P_Solder_Combo
- TOF4: renamed from IR4; value Conn_01x06 -> TOF_I2C; footprint chu_main:GP2Y0E03 -> chu_main:SH1.0_4P_Solder_Combo
- TOF5: renamed from IR5; value Conn_01x06 -> TOF_I2C; footprint chu_main:GP2Y0E03 -> chu_main:SH1.0_4P_Solder_Combo
- U1: value Pico -> PiPico_No_SWD; footprint chu_main:RPi_Pico_SMD_Pins_Strip -> chu_main:RPi_Pico_SMD_Pins_No_SWD
- moved PN532 8.89 mm to (126.6, 133.5), turned to -90 degrees
- moved TOF2 8.06 mm to (178.2, 143.1), turned to -90 degrees
- moved TOF5 8.06 mm to (314.2, 143.1), turned to 90 degrees
- moved TOF1 7.00 mm to (114.2, 143.1), turned to -90 degrees
- moved R12 4.00 mm to (323.4, 150.9)
- moved R13 4.00 mm to (325.3, 150.9)
- moved TOF3 3.61 mm to (252.2, 138.1), turned to -90 degrees
- moved R5 3.30 mm to (185.9, 142.5)
- moved R4 3.20 mm to (187.6, 142.5)
- moved TOF4 2.15 mm to (247.0, 148.1), turned to 90 degrees
- moved C8 1.36 mm to (192.2, 139.6)
- moved R2 0.89 mm to (86.0, 116.6)
- moved R1 0.40 mm to (85.4, 118.7)
Connections:
- D1 pad I: Net-(D1-PadI) -> Net-(D1-In)
- PN532 pad 1: /SCL_1 -> GND
- PN532 pad 3: +3V3 -> /SCL_1
- PN532 pad 4: GND -> +3V3
- TOF1 pad 1: +3V3 -> GND
- TOF1 pad 2: GND -> /SDA_1
- TOF1 pad 3: +3V3 -> /SCL_1
- TOF2 pad 1: +3V3 -> GND
- TOF2 pad 2: GND -> /SDA_2
- TOF2 pad 3: +3V3 -> /SCL_2
- TOF3 pad 1: +3V3 -> GND
- TOF3 pad 2: GND -> /SDA_3
- TOF3 pad 3: +3V3 -> /SCL_3
- TOF4 pad 1: +3V3 -> GND
- TOF4 pad 2: GND -> /SDA_4
- TOF4 pad 3: +3V3 -> /SCL_4
- TOF5 pad 1: +3V3 -> GND
- TOF5 pad 2: GND -> /SDA_5
- TOF5 pad 3: +3V3 -> /SCL_5
- U1 pad 17: unconnected-(U1-Pad17) -> Net-(SW1-A)
- U1 pad 19: unconnected-(U1-Pad19) -> Net-(SW2-A)
- U1 pad 20: unconnected-(U1-Pad20) -> Net-(SW3-A)
- U1 pad 39: unconnected-(U1-Pad39) -> +5V
- U1 pad 4: Net-(R3-Pad2) -> Net-(D1-In)
- U1 pad 40: +5V -> VBUS
- USB1 pad 11: +5V -> VBUS
- USB1 pad 13: unconnected-(USB1-Pad13) -> GND
- USB1 pad 2: +5V -> VBUS
Routing:
- net Net-(SW3-A): track 0.00 -> 272.3 mm
- net Net-(SW2-A): track 0.00 -> 267.2 mm
- net Net-(SW1-A): track 0.00 -> 264.3 mm
- net GND: track 167.7 -> 266.1 mm, vias 48 -> 54
- net Net-(D1-In): track 0.00 -> 81.8 mm, vias 0 -> 1
- net +3V3: track 444.1 -> 510.7 mm
- net VBUS: track 0.00 -> 50.4 mm, vias 0 -> 3
- net Net-(R3-Pad2): track 50.0 -> 0.00 mm
- net Net-(D1-PadI): track 35.6 -> 0.00 mm, vias 1 -> 0
- net /SDA_2: track 17.8 -> 35.1 mm
- net unconnected-(USB1-Pad13): track 17.0 -> 0.00 mm
- net /SDA_1: track 92.6 -> 109.6 mm
- net /SCL_2: track 14.9 -> 30.7 mm
- net /SCL_1: track 89.4 -> 105.0 mm
- net +5V: track 761.3 -> 747.8 mm, vias 14 -> 11
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Other:
- outline, holes or cut-outs redrawn
- board text added: "Chu Pico V1.6"
- board text added: "G D C V"
- board text added: "V C D G"
- board text added: "V V"
- board text removed: "Chu Pico V1.5"

Commit message: PCB v1.61 (fix TOF silkscreen marks)
Other:
- board text added: "Chu Pico V1.61"
- board text added: "D C"
- board text added: "G V"
- board text added: "V C D V"
- board text added: "V D C V"
- board text added: "V G"
- board text removed: "Chu Pico V1.6"
- board text removed: "G D C V"
- board text removed: "V C D G"
- board text removed: "V V"
Changed lines of the file:
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@@
 		(tags "connector JST SH horizontal")
 		(property "Reference" "TOF1"
-			(at 5.3 0 360)
+			(at 5.3 0 0)
 			(layer "F.SilkS")
 			(effects
@@
 		)
 		(property "Field4" "PN532"
-			(at -1 5.62 0)
+			(at -3.55 6.53 0)
 			(layer "F.SilkS")
 			(effects
@@
 		(fp_arc
 			(start -1.800001 0.379999)
-			(mid -2.409033 0.362746)
+			(mid -2.409036 0.362746)
 			(end -2.549998 -0.23)
 			(stroke
@@
 		(fp_arc
 			(start -1.800001 0.379999)
-			(mid -2.409033 0.362746)
+			(mid -2.409036 0.362746)
 			(end -2.549998 -0.23)
 			(stroke
@@
 		(fp_arc
 			(start -1.800001 0.379999)
-			(mid -2.409033 0.362746)
+			(mid -2.409036 0.362746)
 			(end -2.549998 -0.23)
 			(stroke
@@
 		(layer "Edge.Cuts")
 	)
-	(gr_text "V\n\n\nV"
-		(at 250.196 151.674 0)
+	(gr_text " V\nC\nD\n V"
+		(at 249.796 151.674 0)
 		(layer "F.SilkS")
 		(effects
 			(font
-				(size 1.15 1.4)
+				(size 1.2 1.4)
 				(thickness 0.2)
 				(bold yes)
@@
 		)
 	)
-	(gr_text "V\n\n\nV"
-		(at 309.296 146.474 0)
+	(gr_text " V\nC\nD\n V"
+		(at 316.996 146.674 0)
 		(layer "F.SilkS")
 		(effects
 			(font
-				(size 1.15 1.4)
+				(size 1.2 1.4)
 				(thickness 0.2)
 				(bold yes)
@@
 		)
 	)
-	(gr_text "V\n C\n D\nG"
-		(at 240.996 151.574 0)
+	(gr_text "V\n\n\nG"
+		(at 241.996 151.774 0)
 		(layer "F.SilkS")
 		(effects
 			(font
-				(size 1.15 1.4)
+				(size 1.2 1.4)
 				(thickness 0.2)
 				(bold yes)
@@
 		)
 	)
-	(gr_text "V\n\n\nV"
-		(at 247.496 141.574 0)
+	(gr_text "D\nC"
+		(at 122.296 135.174 0)
 		(layer "F.SilkS")
 		(effects
 			(font
-				(size 1.15 1.4)
+				(size 1.2 1.4)
 				(thickness 0.2)
 				(bold yes)
@@
 		)
 	)
-	(gr_text "V\n\n\nV"
-		(at 109.596 146.574 0)
+	(gr_text "V\n D\n C\nV"
+		(at 108.796 146.674 0)
 		(layer "F.SilkS")
 		(effects
 			(font
-				(size 1.15 1.4)
+				(size 1.2 1.4)
 				(thickness 0.2)
 				(bold yes)
@@
 		)
 	)
-	(gr_text " G\nD\nC\n V"
-		(at 317.096 146.574 0)
+	(gr_text "V\n\n\nG"
+		(at 309.096 146.774 0)
 		(layer "F.SilkS")
 		(effects
 			(font
-				(size 1.15 1.4)
+				(size 1.2 1.4)
 				(thickness 0.2)
 				(bold yes)
@@
 		)
 	)
-	(gr_text " G\nD\nC\n V"
-		(at 129.876 137.234 0)
+	(gr_text " G\n\n\n V"
+		(at 128.996 137.174 0)
 		(layer "F.SilkS")
 		(effects
 			(font
-				(size 1.15 1.4)
+				(size 1.2 1.4)
 				(thickness 0.2)
 				(bold yes)
@@
 		)
 	)
-	(gr_text "V\n\n\nV"
-		(at 173.596 146.574 0)
+	(gr_text "V\n D\n C\nV"
+		(at 172.796 146.674 0)
 		(layer "F.SilkS")
 		(effects
 			(font
-				(size 1.15 1.4)
+				(size 1.2 1.4)
 				(thickness 0.2)
 				(bold yes)
@@
 		)
 	)
-	(gr_text " G\nD\nC\n V"
-		(at 181.096 146.574 0)
+	(gr_text "Chu Pico V1.61"
+		(at 102.376 132.274 0)
 		(layer "F.SilkS")
 		(effects
 			(font
-				(size 1.15 1.4)
+				(size 1.5 1.5)
+				(thickness 0.3)
+			)
+		)
+	)
+	(gr_text "V\n D\n C\nV"
+		(at 246.796 141.674 0)
+		(layer "F.SilkS")
+		(effects
+			(font
+				(size 1.2 1.4)
 				(thickness 0.2)
 				(bold yes)
@@
 		)
 	)
-	(gr_text "Chu Pico V1.6"
-		(at 102.376 132.274 0)
+	(gr_text "G\n\n\nV"
+		(at 117.696 146.674 0)
 		(layer "F.SilkS")
 		(effects
 			(font
-				(size 1.5 1.5)
-				(thickness 0.3)
+				(size 1.2 1.4)
+				(thickness 0.2)
+				(bold yes)
 			)
+			(justify left bottom)
 		)
 	)
-	(gr_text " G\nD\nC\n V"
-		(at 117.446 146.574 0)
+	(gr_text "G\n\n\nV"
+		(at 255.696 141.674 0)
 		(layer "F.SilkS")
 		(effects
 			(font
-				(size 1.15 1.4)
+				(size 1.2 1.4)
 				(thickness 0.2)
 				(bold yes)
@@
 		)
 	)
-	(gr_text " G\nD\nC\n V"
-		(at 255.296 141.474 0)
+	(gr_text "G\n\n\nV"
+		(at 181.696 146.574 0)
 		(layer "F.SilkS")
 		(effects
 			(font
-				(size 1.15 1.4)
+				(size 1.2 1.4)
 				(thickness 0.2)
 				(bold yes)
