File: PCB/main/chu_main.kicad_sch (KiCad schematic)
At the start: 112 parts, among them J1 Conn_01x04, K1 Conn_01x01_Female, K10 Conn_01x01_Female, K11 Conn_01x01_Female, K12 Conn_01x01_Female, K13 Conn_01x01_Female, K14 Conn_01x01_Female, K15 Conn_01x01_Female, K16 Conn_01x01_Female, K17 Conn_01x01_Female, K18 Conn_01x01_Female, K19 Conn_01x01_Female, K2 Conn_01x01_Female, K20 Conn_01x01_Female, K21 Conn_01x01_Female, K22 Conn_01x01_Female, K23 Conn_01x01_Female, K24 Conn_01x01_Female, K25 Conn_01x01_Female, K26 Conn_01x01_Female, K27 Conn_01x01_Female, K28 Conn_01x01_Female, K29 Conn_01x01_Female, K3 Conn_01x01_Female, K30 Conn_01x01_Female, K31 Conn_01x01_Female, K32 Conn_01x01_Female, K4 Conn_01x01_Female, K5 Conn_01x01_Female, K6 Conn_01x01_Female, K7 Conn_01x01_Female, K8 Conn_01x01_Female, K9 Conn_01x01_Female, U0 ChuAcrylic, U1 Pico, U2 PCA9548APW, U3 MPR121QR2_BOARD, U4 MPR121QR2_BOARD, U5 MPR121QR2_BOARD, U8 SN74LV1T34DBV, X1 GP2Y0E03_REAL, X2 GP2Y0E03_REAL, X3 GP2Y0E03_REAL, X4 GP2Y0E03_REAL, X5 GP2Y0E03_REAL

Commit message: Chu main PCB v1.6
Parts:
- removed IR1, IR2, IR3, IR4, IR5: Conn_01x06, chu_main:GP2Y0E03, symbol Connector_Generic:Conn_01x06
- removed J1: Conn_01x04, chu_main:PN532, symbol Connector_Generic:Conn_01x04
- removed R3: 10, Resistor_SMD:R_0603_1608Metric, symbol Device:R_Small
- removed U1: Pico, chu_main:RPi_Pico_SMD_Pins_Strip, symbol MCU_RaspberryPi_and_Boards:Pico
- removed U8: SN74LV1T34DBV, chu_main:SOT-23-5_Jumper, symbol Logic_LevelTranslator:SN74LV1T34DBV
- added PN532, TOF1, TOF2, TOF3, TOF4, TOF5: TOF_I2C, chu_main:SH1.0_4P_Solder_Combo, symbol chu_main:TOF_I2C
- added SW1, SW2, SW3: SPST_EVQP4, chu_main:SW_EVQ-P46B3M, symbol chu_main:SPST_EVQP4
- added U1: PiPico_No_SWD, chu_main:RPi_Pico_SMD_Pins_No_SWD, symbol chu_main:PiPico_No_SWD
- R1, R10, R11, R12, R13, R2, R4, R5, R6, R7, R8, R9: footprint Resistor_SMD:R_0603_1608Metric -> Resistor_SMD:R_0603_1608Metric_Pad0.98x0.95mm_HandSolder
Connections:
- net +3V3: now also PN532.4 (Pin_4), TOF1.4 (Pin_4), TOF1.MP, TOF2.4 (Pin_4), TOF2.MP, TOF3.4 (Pin_4), TOF3.MP, TOF4.4 (Pin_4), TOF4.MP, TOF5.4 (Pin_4), TOF5.MP, U1.36 (3V3)
- net +5V: now also U1.39 (VSYS); no longer USB1.11 (VBUS), USB1.2 (VBUS)
- net GND: now also USB1.13 (SHIELD), PN532.1 (Pin_1), SW1.2 (B), SW1.MP, SW2.2 (B), SW2.MP, SW3.2 (B), SW3.MP, TOF1.1 (Pin_1), TOF2.1 (Pin_1), TOF3.1 (Pin_1), TOF4.1 (Pin_1), TOF5.1 (Pin_1), U1.13 (GND), U1.18 (GND), U1.23 (GND), U1.28 (GND), U1.3 (GND), U1.33 (AGND), U1.38 (GND), U1.8 (GND)
- net SCL: now also U1.22 (GPIO17)
- net SCL_1: now also PN532.3 (Pin_3), TOF1.3 (Pin_3)
- net SCL_2: now also TOF2.3 (Pin_3)
- net SCL_3: now also TOF3.3 (Pin_3)
- net SCL_4: now also TOF4.3 (Pin_3)
- net SCL_5: now also TOF5.3 (Pin_3)
- net SDA: now also U1.21 (GPIO16)
- net SDA_1: now also PN532.2 (Pin_2), TOF1.2 (Pin_2)
- net SDA_2: now also TOF2.2 (Pin_2)
- net SDA_3: now also TOF3.2 (Pin_2)
- net SDA_4: now also TOF4.2 (Pin_2)
- net SDA_5: now also TOF5.2 (Pin_2)
- net at U2.3 (~{RESET}): now also U1.25 (GPIO19)
- net at USB1.5 (DN2), USB1.7 (DN1): now also U1.TP2 (USB1)
- net at USB1.6 (DP1), USB1.8 (DP2): now also U1.TP3 (USB2)
- net at D1.I (In): now also U1.4 (GPIO2)
- new net: SW1.1 (A), U1.17 (GPIO13)
- new net: SW2.1 (A), U1.19 (GPIO14)
- new net: SW3.1 (A), U1.20 (GPIO15)
- new net VBUS: U1.40 (VBUS), USB1.11 (VBUS), USB1.2 (VBUS)
- no-connect marks 41 -> 35
Other:
- moved on the sheet: R10, R11, R12, R13, R4, R5, R6, R7, R8, R9
